File: 75%/75%.kicad_pcb (KiCad board)
At the start: 2 copper layers, 326.7 x 135.4 mm, 167 parts, among them U1 ATmega32U4-A

Commit message: updated the via
Routing:
- net Column 14: track 121.4 -> 120.7 mm, vias 2 -> 1

Commit message: quick fixes
Connections:
- U1 pad 1: unconnected-(U1-PE6-Pad1) -> Column 10
- U1 pad 33: Column 10 -> Net-(U1-~{HWB}/PE2)
Routing:
- net Column 10: track 209.8 -> 227.2 mm, vias 0 -> 1
- net Column 1: track 424.0 -> 429.8 mm
- net Column 0: track 449.7 -> 455.0 mm
- net Column 5: track 312.4 -> 314.9 mm
- net Column 6: track 310.6 -> 313.1 mm
- net Column 4: track 335.2 -> 337.7 mm
- net Column 3: track 356.0 -> 358.5 mm
- net Column 2: track 401.5 -> 403.8 mm
- net Column 7: track 254.8 -> 256.8 mm
- net Net-(U1-GND-Pad15): track 26.9 -> 25.3 mm, vias 2 -> 0
- net Column 9: track 211.6 -> 212.7 mm
- net Column 8: track 234.6 -> 235.7 mm
- net Net-(U1-VCC-Pad14): track 14.1 -> 14.4 mm, vias 0 -> 2

Commit message: latest
Parts:
- added C1: 1uF, Capacitor_SMD:C_0805_2012Metric, B.Cu at (368.6, 83.0)
- added C2: 10uF, Capacitor_SMD:C_0805_2012Metric, B.Cu at (361.8, 96.8)
- added C3: 1uF, Capacitor_SMD:C_0805_2012Metric, B.Cu at (358.5, 96.1)
- added C4: 100nF, Capacitor_SMD:C_0805_2012Metric, B.Cu at (366.8, 73.8)
- added C5: 100nF, Capacitor_SMD:C_0805_2012Metric, B.Cu at (368.5, 78.9)
- added J2: USB_C_Receptacle, Connector_USB:USB_C_Receptacle_GCT_USB4105-xx-A_16P_TopMnt_Horizontal, B.Cu at (369.5, 93.2)
- added R1: 10k, Resistor_SMD:R_0805_2012Metric, B.Cu at (352.3, 95.6)
- added R3: 22ohm, Resistor_SMD:R_0805_2012Metric, F.Cu at (348.0, 96.6)
- added R4: 22ohm, Resistor_SMD:R_0805_2012Metric, F.Cu at (349.9, 96.6)
- added R5: 5.1k, Resistor_SMD:R_0805_2012Metric, B.Cu at (370.8, 85.6)
- added R6: 5.1k, Resistor_SMD:R_0805_2012Metric, B.Cu at (361.1, 93.1)
- added SW1: SW_Push, Button_Switch_THT:SW_PUSH-12mm, B.Cu at (358.2, 165.6)
Connections:
- U1 pad 13: unconnected-(U1-~{RESET}-Pad13) -> Net-(U1-~{RESET})
- U1 pad 14: Net-(U1-VCC-Pad14) -> VBUS
- U1 pad 15: Net-(U1-GND-Pad15) -> GND
- U1 pad 2: unconnected-(U1-UVCC-Pad2) -> VBUS
- U1 pad 23: Net-(U1-GND-Pad15) -> GND
- U1 pad 24: Net-(U1-AVCC-Pad24) -> VBUS
- U1 pad 3: unconnected-(U1-D--Pad3) -> Net-(U1-D-)
- U1 pad 33: Net-(U1-~{HWB}/PE2) -> unconnected-(U1-~{HWB}/PE2-Pad33)
- U1 pad 34: Net-(U1-VCC-Pad14) -> VBUS
- U1 pad 35: Net-(U1-GND-Pad15) -> GND
- U1 pad 4: unconnected-(U1-D+-Pad4) -> Net-(U1-D+)
- U1 pad 43: Net-(U1-GND-Pad15) -> GND
- U1 pad 44: Net-(U1-AVCC-Pad24) -> VBUS
- U1 pad 5: unconnected-(U1-UGND-Pad5) -> GND
- U1 pad 6: unconnected-(U1-UCAP-Pad6) -> Net-(U1-UCAP)
- U1 pad 7: unconnected-(U1-VBUS-Pad7) -> VBUS
Routing:
- net GND: track 0.00 -> 205.4 mm, vias 0 -> 4
- net Net-(U1-~{RESET}): track 0.00 -> 103.2 mm, vias 0 -> 3
- net VBUS: track 0.00 -> 79.8 mm, vias 0 -> 8
- net Net-(U1-GND-Pad15): track 25.3 -> 0.00 mm
- net D-: track 0.00 -> 24.2 mm, vias 0 -> 1
- net D+: track 0.00 -> 23.7 mm, vias 0 -> 1
- net Net-(U1-D+): track 0.00 -> 21.1 mm, vias 0 -> 1
- net Net-(U1-D-): track 0.00 -> 20.7 mm, vias 0 -> 1
- net Net-(U1-UCAP): track 0.00 -> 15.1 mm, vias 0 -> 2
- net Net-(U1-AVCC-Pad24): track 14.7 -> 0.00 mm, vias 2 -> 0
- net Net-(U1-VCC-Pad14): track 14.4 -> 0.00 mm, vias 2 -> 0
- net Net-(J2-CC1): track 0.00 -> 8.48 mm
- net Net-(J2-CC2): track 0.00 -> 5.05 mm
