File: 75%/75%.kicad_sch (KiCad schematic)
At the start: 168 parts, among them J1 USB_C_Receptacle, U1 ATmega32U4-A

Commit message: quick fixes
Parts:
- removed J1: USB_C_Receptacle, symbol Connector:USB_C_Receptacle
Connections:
- net Column 10: now also U1.1 (PE6); no longer U1.33 (~{HWB}/PE2)
- net VBUS: now reaches U1.14 (VCC), U1.34 (VCC)
- net VBUS: now also U1.2 (UVCC), U1.24 (AVCC), U1.44 (AVCC), U1.7 (VBUS)
- net GND: now reaches U1.15 (GND), U1.23 (GND), U1.35 (GND), U1.43 (GND)
- net GND: now also U1.5 (UGND)
- net D-: now reaches U1.3 (D-)
- net D+: now reaches U1.4 (D+)
Other:
- added sheet Data (untitled.kicad_sch)

Commit message: latest
Parts:
- added C1, C3: 1uF, Capacitor_SMD:C_0805_2012Metric, symbol Device:C_Small
- added C2: 10uF, Capacitor_SMD:C_0805_2012Metric, symbol Device:C_Small
- added C4, C5: 100nF, Capacitor_SMD:C_0805_2012Metric, symbol Device:C_Small
- added J2: USB_C_Receptacle, Connector_USB:USB_C_Receptacle_GCT_USB4105-xx-A_16P_TopMnt_Horizontal, symbol Connector:USB_C_Receptacle
- added R1: 10k, Resistor_SMD:R_0805_2012Metric, symbol Device:R_Small
- added R3, R4: 22ohm, Resistor_SMD:R_0805_2012Metric, symbol Device:R_Small
- added R5, R6: 5.1k, Resistor_SMD:R_0805_2012Metric, symbol Device:R_Small
- added SW1: SW_Push, Button_Switch_THT:SW_PUSH-12mm, symbol Switch:SW_Push
Connections:
- net D+: now also J2.A6 (D+), J2.B6 (D+), R3.1; no longer U1.4 (D+)
- net D-: now also J2.A7 (D-), J2.B7 (D-), R4.1; no longer U1.3 (D-)
- net GND: now also C1.2, C2.1, C3.2, C4.2, C5.2, J2.A1 (GND), J2.A12 (GND), J2.B1 (GND), J2.B12 (GND), J2.S1 (SHIELD), R5.2, R6.2, SW1.1
- net VBUS: now also C2.2, C3.1, C4.1, C5.1, J2.A4 (VBUS), J2.A9 (VBUS), J2.B4 (VBUS), J2.B9 (VBUS), R1.2
- net at U1.13 (~{RESET}): now also R1.1, SW1.2
- net at U1.6 (UCAP): now also C1.1
- new net: J2.A5 (CC1), R5.1
- new net: J2.B5 (CC2), R6.1
- new net: R4.2, U1.3 (D-)
- new net: R3.2, U1.4 (D+)
- no-connect marks 0 -> 17
Other:
- removed sheet Data
